File: EGPad.kicad_pcb (KiCad board)
At the start: 2 copper layers, 111.1 x 133.3 mm, 67 parts, among them M2 MountingHole_2mm, SW1 Rotary_Encoder_Switch, SW2 Rotary_Encoder_Switch, SW3 Rotary_Encoder_Switch, U1 ProMicro

Commit message: Polished labels, added gerber file
Routing:
- net Net-(D15-Pad2): track 35.8 -> 34.7 mm
